Commit message: Imported .stl models

File: src/arm_4dof/urdf/arm.urdf (robot description, URDF)
Before this commit: robot my_4dof_arm, 6 links, 5 joints
Links:
- added link end_effector; visual mesh filename=package://arm_4dof/meshes/end_effector.STL scale=1 1 1
- link base_link: geometry visual mesh filename=package://arm_4dof/meshes/base.STL scale=1 1 1
- link base_rotate_link: geometry visual mesh filename=package://arm_4dof/meshes/rotate_link.STL scale=1 1 1
- link elbow_link: geometry visual mesh filename=package://arm_4dof/meshes/elbow_link.STL scale=1 1 1
- link shoulder_link: geometry visual mesh filename=package://arm_4dof/meshes/shoulder_link.STL scale=1 1 1
- link wrist_link: geometry visual mesh filename=package://arm_4dof/meshes/wrist_link.STL scale=1 1 1
Joints:
- added joint endeffector: type fixed, parent wrist_link, child end_effector, origin xyz=0 0 0.425 rpy=0 0 0
- joint base_rotate_joint: origin xyz=0 0 0.1 rpy=0 0 0 -> xyz=0 0 0.05 rpy=0 0 0
- joint elbow_joint: origin xyz=0 0 0.4 rpy=0 0 0 -> xyz=0 0 1.3 rpy=0 0 0
- joint shoulder_joint: origin xyz=0 0 0 rpy=0 0 0 -> xyz=0 0 0.65 rpy=0 0 0
- joint wrist_joint: origin xyz=0 0 0.4 rpy=0 0 0 -> xyz=0 0 0.92 rpy=0 0 0
